File: Hunter_Keyboard_Schematic/Husky_Hunter_Keyboard.kicad_sch (KiCad schematic)
At the start: 59 parts, among them J1 Conn_01x17_Socket, SW1 SHIFT_L, SW10 COMMA, SW11 PERIOD, SW12 FWD_SLASH, SW13 TAB, SW14 SHIIFT_R, SW15 CTL, SW16 A, SW17 S, SW18 D, SW19 F, SW2 Z, SW20 G, SW21 H, SW22 J, SW23 K, SW24 L, SW25 SEMI_COLON, SW26 QUOTE, SW27 CURS_DOWN, SW28 DEL, SW29 ENTER, SW3 X, SW30 Q, SW31 W, SW32 E, SW33 R, SW34 T, SW35 Y, SW36 U, SW37 I, SW38 O, SW39 P, SW4 C, SW40 SQ_BRACKET, SW41 CURS_LEFT, SW42 INS, SW43 CURS_RIGHT, SW44 ONE, SW45 TWO, SW46 THREE, SW47 FOUR, SW48 FIVE, SW49 SIX, SW5 V, SW50 SEVEN, SW51 EIGHT, SW52 NINE, SW53 ZERO, SW54 MINUS, SW55 EQUALS, SW56 CURS_UP, SW57 ESC, SW58 POWER, SW6 B, SW7 N, SW8 M, SW9 SPACE

Commit message: PCB design created for testing
Parts:
- added H1, H2, H3, H4: MountingHole, MountingHole:MountingHole_3.2mm_M3_Pad, symbol Mechanical:MountingHole
- J1: footprint (none) -> Connector_PinSocket_2.54mm:PinSocket_1x17_P2.54mm_Horizontal
- SW1, SW10, SW11, SW12, SW13, SW14, SW15, SW16, SW17, SW18, SW19, SW2, SW20, SW21, SW22, SW23, SW24, SW25, SW26, SW27, SW28, SW29, SW3, SW30, SW31, SW32, SW33, SW34, SW35, SW36, SW37, SW38, SW39, SW4, SW40, SW41, SW42, SW43, SW44, SW45, SW46, SW47, SW48, SW49, SW5, SW50, SW51, SW52, SW53, SW54, SW55, SW56, SW57, SW6, SW7, SW8, SW9: footprint (none) -> Button_Switch_Keyboard:SW_Cherry_MX_1.00u_PCB
- SW58: footprint (none) -> Clueless_Engineer:Switch_Tactile_6mm
Other:
- company: https://youtube.com/@brfff -> Brett Hallen
- title: Husky Hunter Keyboard -> Husky Hunter External Keyboard
